File: hardware/console.kicad_pcb (KiCad board)
At the start: 2 copper layers, 44 x 72 mm, 47 parts, among them J1 USB-C_Module, J3 SWD, J4 UART, J5 LiPo_140mAh, SW1 SW_PUSH, SW2 SW_PUSH, SW3 SW_PUSH, SW4 SW_PUSH, SW5 SW_PUSH, SW6 SW_PUSH, SW7 SW_POWER, SW8 SW_PUSH, SW9 SW_PUSH, U1 STM32G070CBT6, U2 XC6206P332MR, U3 TP4054

Commit message: hardware is done, this is what was sent
Other:
- board text added: "13/08/2026"
Changed lines of the file:
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@@
 			(pinfunction "VSS_7")
 			(pintype "power_in")
+			(zone_connect 2)
 		)
 		(pad "8" smd roundrect
@@
 			)
 		)
-		(attr exclude_from_bom)
+		(attr exclude_from_pos_files exclude_from_bom)
 		(duplicate_pad_numbers_are_jumpers no)
 		(fp_circle
@@
 			)
 		)
-		(attr through_hole exclude_from_bom)
+		(attr through_hole exclude_from_pos_files exclude_from_bom)
 		(duplicate_pad_numbers_are_jumpers no)
 		(fp_line
@@
 			)
 		)
-		(attr through_hole exclude_from_bom)
+		(attr through_hole exclude_from_pos_files exclude_from_bom)
 		(duplicate_pad_numbers_are_jumpers no)
 		(fp_line
@@
 			)
 		)
-		(attr through_hole exclude_from_pos_files)
+		(attr through_hole exclude_from_pos_files exclude_from_bom)
 		(duplicate_pad_numbers_are_jumpers no)
 		(fp_rect
@@
 		)
 	)
+	(gr_text "13/08/2026"
+		(at 109.75 90.25 0)
+		(layer "B.SilkS")
+		(effects
+			(font
+				(size 1 1)
+				(thickness 0.15)
+			)
+			(justify left bottom mirror)
+		)
+	)
 	(gr_text "Board Rev 1.0"
 		(at 110 92.5 0)
@@
 	)
 	(segment
+		(start 107.288138 57.711863)
+		(end 107 58)
+		(width 0.25)
+		(layer "F.Cu")
+		(net "GND")
+	)
+	(segment
+		(start 84.393804 76.92)
+		(end 84.1 76.92)
+		(width 0.25)
+		(layer "F.Cu")
+		(net "GND")
+	)
+	(segment
+		(start 84.598804 77.125)
+		(end 84.393804 76.92)
+		(width 0.25)
+		(layer "F.Cu")
+		(net "GND")
+	)
+	(segment
+		(start 84.719504 77.25)
+		(end 86.3375 77.25)
+		(width 0.25)
+		(layer "F.Cu")
+		(net "GND")
+	)
+	(segment
+		(start 82.8346 75.0546)
+		(end 83.217844 75.0546)
+		(width 0.25)
+		(layer "F.Cu")
+		(net "GND")
+	)
+	(segment
 		(start 73.48 58.5)
 		(end 73.3297 58.0231)
@@
 	)
 	(segment
-		(start 106.93 58)
-		(end 107.43 58)
+		(start 82.735 74.955)
+		(end 82.8346 75.0546)
 		(width 0.25)
 		(layer "F.Cu")
@@
 	)
 	(segment
-		(start 84.1 79.12)
-		(end 83.6231 79.2704)
+		(start 82.455 74.675)
+		(end 82.46649 74.675)
 		(width 0.25)
 		(layer "F.Cu")
@@
 	)
 	(segment
-		(start 82.1 76.825)
-		(end 82.483 77.1464)
+		(start 107 58)
+		(end 106.93 58)
 		(width 0.25)
 		(layer "F.Cu")
@@
 	)
 	(segment
-		(start 84.1 76.92)
-		(end 84.7108 77.1423)
+		(start 82.57351 77.13859)
+		(end 82.41359 77.13859)
+		(width 0.25)
+		(layer "F.Cu")
+		(net "GND")
+	)
+	(segment
+		(start 82.5821 77.13)
+		(end 82.57351 77.13859)
 		(width 0.25)
 		(layer "F.Cu")
@@
 	)
 	(segment
-		(start 86.3375 77.25)
-		(end 85.4 77.25)
+		(start 84.598804 77.1293)
+		(end 84.719504 77.25)
+		(width 0.25)
+		(layer "F.Cu")
+		(net "GND")
+	)
+	(segment
+		(start 83.841136 79.12)
+		(end 83.481899 79.479237)
+		(width 0.25)
+		(layer "F.Cu")
+		(net "GND")
+	)
+	(segment
+		(start 84.598804 77.1293)
+		(end 84.598804 77.125)
+		(width 0.25)
+		(layer "F.Cu")
+		(net "GND")
+	)
+	(segment
+		(start 82.41359 77.13859)
+		(end 82.1 76.825)
 		(width 0.25)
 		(layer "F.Cu")
@@
 	)
 	(segment
+		(start 82.46649 74.675)
+		(end 82.735 74.94351)
+		(width 0.25)
+		(layer "F.Cu")
+		(net "GND")
+	)
+	(segment
+		(start 84.1 79.12)
+		(end 83.841136 79.12)
+		(width 0.25)
+		(layer "F.Cu")
+		(net "GND")
+	)
+	(segment
 		(start 82.1 74.32)
-		(end 83.2807 75.0722)
+		(end 82.455 74.675)
 		(width 0.25)
 		(layer "F.Cu")
@@
 	)
 	(segment
-		(start 85.4 77.25)
-		(end 84.7108 77.1423)
+		(start 82.735 74.94351)
+		(end 82.735 74.955)
 		(width 0.25)
 		(layer "F.Cu")
@@
 	(via
 		(at 73.3297 58.0231)
-		(size 0.5)
+		(size 0.6)
 		(drill 0.3)
 		(layers "F.Cu" "B.Cu")
@@
 	(via
 		(at 83.7701 72.8489)
-		(size 0.5)
+		(size 0.6)
 		(drill 0.3)
 		(layers "F.Cu" "B.Cu")
@@
 	(via
 		(at 99.3285 65.317)
-		(size 0.5)
+		(size 0.6)
 		(drill 0.3)
 		(layers "F.Cu" "B.Cu")
@@
 	)
 	(via
-		(at 83.2807 75.0722)
-		(size 0.5)
+		(at 83.217844 75.0546)
+		(size 0.6)
 		(drill 0.3)
 		(layers "F.Cu" "B.Cu")
@@
 	(via
 		(at 76.2187 52.0381)
-		(size 0.5)
+		(size 0.6)
 		(drill 0.3)
 		(layers "F.Cu" "B.Cu")
@@
 	)
 	(via
-		(at 84.7108 77.1423)
-		(size 0.5)
+		(at 84.598804 77.1293)
+		(size 0.6)
 		(drill 0.3)
 		(layers "F.Cu" "B.Cu")
@@
 	)
 	(via
-		(at 82.483 77.1464)
-		(size 0.5)
+		(at 82.5821 77.13)
+		(size 0.6)
 		(drill 0.3)
 		(layers "F.Cu" "B.Cu")
@@
 	)
 	(via
-		(at 107.43 58)
-		(size 0.5)
+		(at 107.288138 57.711863)
+		(size 0.6)
 		(drill 0.3)
 		(layers "F.Cu" "B.Cu")
@@
 	)
 	(via
-		(at 83.6231 79.2704)
-		(size 0.5)
+		(at 83.481899 79.479237)
+		(size 0.6)
 		(drill 0.3)
 		(layers "F.Cu" "B.Cu")
