File: hardware/console.kicad_sch (KiCad schematic)
At the start: 45 parts, among them J1 USB-C_Module, J3 SWD, J4 UART, J5 LiPo_140mAh, SW1 SW_PUSH, SW2 SW_PUSH, SW3 SW_PUSH, SW4 SW_PUSH, SW5 SW_PUSH, SW6 SW_PUSH, SW7 SW_POWER, SW8 SW_PUSH, SW9 SW_PUSH, U1 STM32G070CBT6, U2 XC6206P332MR, U3 TP4054

Commit message: fix battery connector
Parts:
- J5: footprint Connector_JST:JST_PH_B2B-PH-K_1x02_P2.00mm_Vertical -> Connector_JST:JST_PH_S2B-PH-K_1x02_P2.00mm_Horizontal
Changed lines of the file:
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@@
 			)
 		)
-		(property "Footprint" "Connector_JST:JST_PH_B2B-PH-K_1x02_P2.00mm_Vertical"
+		(property "Footprint" "Connector_JST:JST_PH_S2B-PH-K_1x02_P2.00mm_Horizontal"
 			(at 105.41 34.29 0)
 			(hide yes)
@@
 			)
 		)
-		(property "Description" "JST PH-compatible 2.00mm 2-pin battery connector, vertical THT"
+		(property "Description" "JST PH-compatible 2.00mm 2-pin battery connector, side-entry (horizontal) THT"
 			(at 105.41 34.29 0)
 			(hide yes)

Commit message: change buzzer
Parts:
- added TH1, TH2: ToolingHole, console:TOOL-NPTH-D1.152, symbol Mechanical:MountingHole
- DS1: now in the parts list
- LS1: value HNR-1207PA6.5 -> PS1240P02BT; footprint console:BUZ-TH_BD12.5-P6.50-D0.9 -> Buzzer_Beeper:Buzzer_TDK_PS1240P02BT_D12.2mm_H6.5mm; LCSC C22387765 -> C76871; MPN HNR-1207PA6.5 -> PS1240P02BT; Manufacturer (none) -> TDK
Other:
- note added: "Needed for pcba"
- moved on the sheet: H1, TP5, TP6, TP7
Changed lines of the file:
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@@
 		)
 	)
+	(text "Needed for pcba"
+		(exclude_from_sim no)
+		(at 274.828 143.256 0)
+		(effects
+			(font
+				(size 1.27 1.27)
+			)
+		)
+	)
 	(text "Power Supply"
 		(exclude_from_sim no)
@@
 	)
 	(label "VBAT_SENSE"
-		(at 254 133.35 0)
+		(at 247.65 135.89 0)
 		(effects
 			(font
@@
 	)
 	(label "VBAT_LIPO"
-		(at 254 125.73 0)
+		(at 247.65 128.27 0)
 		(effects
 			(font
@@
 	)
 	(label "VBAT_SW"
-		(at 254 129.54 0)
+		(at 247.65 132.08 0)
 		(effects
 			(font
@@
 	)
 	(symbol
+		(lib_id "Mechanical:MountingHole")
+		(at 274.32 147.32 0)
+		(unit 1)
+		(body_style 1)
+		(exclude_from_sim no)
+		(in_bom no)
+		(on_board yes)
+		(in_pos_files no)
+		(dnp no)
+		(property "Reference" "TH2"
+			(at 274.32 152.4 0)
+			(show_name no)
+			(do_not_autoplace no)
+			(effects
+				(font
+					(size 1.27 1.27)
+				)
+			)
+		)
+		(property "Value" "ToolingHole"
+			(at 274.32 150.495 0)
+			(show_name no)
+			(do_not_autoplace no)
+			(effects
+				(font
+					(size 1.27 1.27)
+				)
+			)
+		)
+		(property "Footprint" "console:TOOL-NPTH-D1.152"
+			(at 274.32 147.32 0)
+			(hide yes)
+			(show_name no)
+			(do_not_autoplace no)
+			(effects
+				(font
+					(size 1.27 1.27)
+				)
+			)
+		)
+		(property "Datasheet" ""
+			(at 274.32 147.32 0)
+			(hide yes)
+			(show_name no)
+			(do_not_autoplace no)
+			(effects
+				(font
+					(size 1.27 1.27)
+				)
+			)
+		)
+		(property "Description" "JLCPCB assembly tooling hole, NPTH Ø1.152 mm"
+			(at 274.32 147.32 0)
+			(hide yes)
+			(show_name no)
+			(do_not_autoplace no)
+			(effects
+				(font
+					(size 1.27 1.27)
+				)
+			)
+		)
+		(instances
+			(project "console"
+				(path "/a286ee18-4788-4879-90da-91d936bf6259"
+					(reference "TH2")
+					(unit 1)
+				)
+			)
+		)
+	)
+	(symbol
 		(lib_id "Connector:TestPoint")
-		(at 254 133.35 90)
+		(at 247.65 135.89 90)
 		(unit 1)
 		(body_style 1)
@@
 		(dnp no)
 		(property "Reference" "TP7"
-			(at 247.396 133.35 90)
+			(at 241.046 135.89 90)
 			(show_name no)
 			(do_not_autoplace no)
@@
 		)
 		(property "Value" "VBAT_SENSE"
-			(at 255.27 133.35 0)
+			(at 248.92 135.89 0)
 			(hide yes)
 			(show_name no)
@@
 		)
 		(property "Footprint" "TestPoint:TestPoint_THTPad_D1.5mm_Drill0.7mm"
-			(at 254 128.27 0)
+			(at 247.65 130.81 0)
 			(hide yes)
 			(show_name no)
@@
 		)
 		(property "Datasheet" ""
-			(at 254 128.27 0)
+			(at 247.65 130.81 0)
 			(hide yes)
 			(show_name no)
@@
 		)
 		(property "Description" "test point"
-			(at 254 133.35 0)
+			(at 247.65 135.89 0)
 			(hide yes)
 			(show_name no)
@@
 		(in_bom yes)
 		(on_board yes)
-		(in_pos_files yes)
+		(in_pos_files no)
 		(dnp no)
 		(property "Reference" "LS1"
@@
 			)
 		)
-		(property "Value" "HNR-1207PA6.5"
+		(property "Value" "PS1240P02BT"
 			(at 270.51 85.09 270)
 			(show_name no)
@@
 			)
 		)
-		(property "Footprint" "console:BUZ-TH_BD12.5-P6.50-D0.9"
+		(property "Footprint" "Buzzer_Beeper:Buzzer_TDK_PS1240P02BT_D12.2mm_H6.5mm"
 			(at 270.51 91.44 0)
 			(hide yes)
@@
 			)
 		)
-		(property "Datasheet" ""
+		(property "Datasheet" "https://product.tdk.com/system/files/dam/doc/product/sw_piezo/sw_piezo/piezo-buzzer/catalog/piezoelectronic_buzzer_ps_en.pdf"
+			(at 270.51 91.44 0)
+			(hide yes)
+			(show_name no)
+			(do_not_autoplace no)
+			(effects
+				(font
+					(size 1.27 1.27)
+				)
+			)
+		)
+		(property "Description" "Piezoelectric passive buzzer, 12.2 mm dia through-hole, 5.0 mm pitch. Resonance 4.0 kHz, 3 Vo-p rated (30 V max), 70 dB @ 10 cm."
 			(at 270.51 91.44 0)
 			(hide yes)
@@
 			)
 		)
-		(property "Description" "Piezoelectric passive buzzer, 12.5 mm dia through-hole, 6.5 mm pitch. Resonance 4000 +/-500 Hz, <=10 mA at 5 Vpp, >=80 dB @ 10 cm."
+		(property "MPN" "PS1240P02BT"
 			(at 270.51 91.44 0)
 			(hide yes)
@@
 			)
 		)
-		(property "MPN" "HNR-1207PA6.5"
+		(property "Manufacturer" "TDK"
 			(at 270.51 91.44 0)
 			(hide yes)
@@
 			)
 		)
-		(property "LCSC" "C22387765"
+		(property "LCSC" "C76871"
 			(at 270.51 91.44 0)
 			(hide yes)
@@
 		(body_style 1)
 		(exclude_from_sim no)
-		(in_bom no)
+		(in_bom yes)
 		(on_board yes)
-		(in_pos_files yes)
+		(in_pos_files no)
 		(dnp no)
 		(property "Reference" "DS1"
@@
 	(symbol
 		(lib_id "Connector:TestPoint")
-		(at 254 125.73 90)
+		(at 247.65 128.27 90)
 		(unit 1)
 		(body_style 1)
@@
 		(dnp no)
 		(property "Reference" "TP5"
-			(at 247.142 125.73 90)
+			(at 240.792 128.27 90)
 			(show_name no)
 			(do_not_autoplace no)
@@
 		)
 		(property "Value" "VBAT_LIPO"
-			(at 257.81 125.73 0)
+			(at 251.46 128.27 0)
 			(hide yes)
 			(show_name no)
@@
 		)
 		(property "Footprint" "TestPoint:TestPoint_THTPad_D1.5mm_Drill0.7mm"
-			(at 254 120.65 0)
+			(at 247.65 123.19 0)
 			(hide yes)
 			(show_name no)
@@
 		)
 		(property "Datasheet" ""
-			(at 254 120.65 0)
+			(at 247.65 123.19 0)
 			(hide yes)
 			(show_name no)
@@
 		)
 		(property "Description" "test point"
-			(at 254 125.73 0)
+			(at 247.65 128.27 0)
 			(hide yes)
 			(show_name no)
@@
 	(symbol
 		(lib_id "Mechanical:MountingHole")
-		(at 240.03 147.32 0)
+		(at 240.03 152.4 0)
 		(unit 1)
 		(body_style 1)
@@
 		(fields_autoplaced yes)
 		(property "Reference" "H1"
-			(at 242.57 146.0499 0)
+			(at 242.57 151.1299 0)
 			(show_name no)
 			(do_not_autoplace no)
@@
 		)
 		(property "Value" "MountingHole"
-			(at 242.57 148.5899 0)
+			(at 242.57 153.6699 0)
 			(show_name no)
 			(do_not_autoplace no)
@@
 		)
 		(property "Footprint" "MountingHole:MountingHole_2.1mm"
-			(at 240.03 147.32 0)
+			(at 240.03 152.4 0)
 			(hide yes)
 			(show_name no)
@@
 		)
 		(property "Datasheet" ""
-			(at 240.03 147.32 0)
+			(at 240.03 152.4 0)
 			(hide yes)
 			(show_name no)
@@
 		)
 		(property "Description" "Mounting Hole without connection"
-			(at 240.03 147.32 0)
+			(at 240.03 152.4 0)
 			(hide yes)
 			(show_name no)
@@
 		(lib_name "TestPoint_1")
 		(lib_id "Connector:TestPoint")
-		(at 254 129.54 90)
+		(at 247.65 132.08 90)
 		(unit 1)
 		(body_style 1)
@@
 		(dnp no)
 		(property "Reference" "TP6"
-			(at 247.396 129.54 90)
+			(at 241.046 132.08 90)
 			(show_name no)
 			(do_not_autoplace no)
@@
 		)
 		(property "Value" "VBAT_SW"
-			(at 255.524 129.54 0)
+			(at 249.174 132.08 0)
 			(hide yes)
 			(show_name no)
@@
 		)
 		(property "Footprint" "TestPoint:TestPoint_THTPad_D1.5mm_Drill0.7mm"
-			(at 254 124.46 0)
+			(at 247.65 127 0)
 			(hide yes)
 			(show_name no)
@@
 		)
 		(property "Datasheet" ""
-			(at 254 124.46 0)
+			(at 247.65 127 0)
 			(hide yes)
 			(show_name no)
@@
 		)
 		(property "Description" "test point"
-			(at 254 129.54 0)
+			(at 247.65 132.08 0)
 			(hide yes)
 			(show_name no)
@@
 					(unit 1)
 				)
+			)
+		)
+	)
+	(symbol
+		(lib_id "Mechanical:MountingHole")
+		(at 274.32 156.21 0)
+		(unit 1)
+		(body_style 1)
+		(exclude_from_sim no)
+		(in_bom no)
+		(on_board yes)
+		(in_pos_files no)
+		(dnp no)
+		(property "Reference" "TH1"
+			(at 274.32 161.29 0)
+			(show_name no)
+			(do_not_autoplace no)
+			(effects
+				(font
+					(size 1.27 1.27)
+				)
+			)
+		)
+		(property "Value" "ToolingHole"
+			(at 274.32 159.385 0)
+			(show_name no)
+			(do_not_autoplace no)
+			(effects
+				(font
+					(size 1.27 1.27)
+				)
+			)
+		)
+		(property "Footprint" "console:TOOL-NPTH-D1.152"
+			(at 274.32 156.21 0)
+			(hide yes)
+			(show_name no)
+			(do_not_autoplace no)
+			(effects
+				(font
+					(size 1.27 1.27)
+				)
+			)
+		)
+		(property "Datasheet" ""
+			(at 274.32 156.21 0)
+			(hide yes)
+			(show_name no)
+			(do_not_autoplace no)
+			(effects
+				(font
+					(size 1.27 1.27)
+				)
+			)
+		)
+		(property "Description" "JLCPCB assembly tooling hole, NPTH Ø1.152 mm"
+			(at 274.32 156.21 0)
+			(hide yes)
+			(show_name no)
+			(do_not_autoplace no)
+			(effects
+				(font
+					(size 1.27 1.27)
+				)
+			)
+		)
+		(instances
+			(project "console"
+				(path "/a286ee18-4788-4879-90da-91d936bf6259"
+					(reference "TH1")
+					(unit 1)
+				)

Commit message: BOM/POS flags
Parts:
- DS1, LS1: now left out of the parts list
Changed lines of the file:
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@@
 		(in_bom no)
 		(on_board yes)
-		(in_pos_files yes)
+		(in_pos_files no)
 		(dnp no)
 		(fields_autoplaced yes)
@@
 		(in_bom no)
 		(on_board yes)
-		(in_pos_files yes)
+		(in_pos_files no)
 		(dnp no)
 		(property "Reference" "J3"
@@
 		(body_style 1)
 		(exclude_from_sim no)
-		(in_bom yes)
+		(in_bom no)
 		(on_board yes)
 		(in_pos_files no)
@@
 		(body_style 1)
 		(exclude_from_sim no)
-		(in_bom yes)
+		(in_bom no)
 		(on_board yes)
 		(in_pos_files no)

Commit message: hardware is done, this is what was sent
Parts:
- J1: now left out of the parts list
Changed lines of the file:
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@@
 		(in_bom no)
 		(on_board yes)
-		(in_pos_files yes)
+		(in_pos_files no)
 		(dnp no)
 		(property "Reference" "J5"
@@
 		(in_bom no)
 		(on_board yes)
-		(in_pos_files yes)
+		(in_pos_files no)
 		(dnp no)
 		(property "Reference" "SW7"
@@
 		(in_bom no)
 		(on_board yes)
-		(in_pos_files yes)
+		(in_pos_files no)
 		(dnp no)
 		(fields_autoplaced yes)
@@
 		(body_style 1)
 		(exclude_from_sim no)
-		(in_bom yes)
+		(in_bom no)
 		(on_board yes)
 		(in_pos_files no)
